Commit message: Create robot.urdf from iiwa14_touch_s_model.urdf.xacro with robot.urdf robot_name:=iiwa and hardware_interface:=PositionJointInterface.

File: urdf/robot.urdf (robot description, URDF)
Before this commit: robot iiwa14, 1 links, 0 joints
Links:
- added link iiwa_link_0, mass 5; collision mesh filename=package://iiwa_description/meshes/iiwa14/collision/link_0.s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; visual mesh filename=package://iiwa_description/meshes/iiwa14/visual/link_0.stl
- added link iiwa_link_1, mass 4; collision mesh filename=package://iiwa_description/meshes/iiwa14/collision/link_1.s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; visual mesh filename=package://iiwa_description/meshes/iiwa14/visual/link_1.stl
- added link iiwa_link_2, mass 4; collision mesh filename=package://iiwa_description/meshes/iiwa14/collision/link_2.s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; visual mesh filename=package://iiwa_description/meshes/iiwa14/visual/link_2.stl
- added link iiwa_link_3, mass 3; collision mesh filename=package://iiwa_description/meshes/iiwa14/collision/link_3.s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; visual mesh filename=package://iiwa_description/meshes/iiwa14/visual/link_3.stl
- added link iiwa_link_4, mass 2.7; collision mesh filename=package://iiwa_description/meshes/iiwa14/collision/link_4.s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; visual mesh filename=package://iiwa_description/meshes/iiwa14/visual/link_4.stl
- added link iiwa_link_5, mass 1.7; collision mesh filename=package://iiwa_description/meshes/iiwa14/collision/link_5.s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; visual mesh filename=package://iiwa_description/meshes/iiwa14/visual/link_5.stl
- added link iiwa_link_6, mass 1.8; collision mesh filename=package://iiwa_description/meshes/iiwa14/collision/link_6.s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; visual mesh filename=package://iiwa_description/meshes/iiwa14/visual/link_6.stl
- added link iiwa_link_7, mass 0.3; collision mesh filename=package://iiwa_description/meshes/iiwa14/collision/link_7.s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; visual mesh filename=package://iiwa_description/meshes/iiwa14/visual/link_7.stl
- added link iiwa_link_ee
- added link iiwa_s_model_connector; collision cylinder length=0.06 radius=0.04; visual cylinder length=0.06 radius=0.04
- added link iiwa_s_model_finger_1; collision mesh filename=package://robotiq_s_model_visualization/meshes/s-model/coll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; visual mesh filename=package://robotiq_s_model_visualization/meshes/s-model/visu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
- added link iiwa_s_model_finger_2; collision mesh filename=package://robotiq_s_model_visualization/meshes/s-model/coll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; visual mesh filename=package://robotiq_s_model_visualization/meshes/s-model/visu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
- added link iiwa_s_model_finger_3; collision mesh filename=package://robotiq_s_model_visualization/meshes/s-model/coll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; visual mesh filename=package://robotiq_s_model_visualization/meshes/s-model/visu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
- added link iiwa_s_model_palm; collision mesh filename=package://robotiq_s_model_visualization/meshes/s-model/coll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; visual mesh filename=package://robotiq_s_model_visualization/meshes/s-model/visu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
Joints:
- added joint iiwa_connector_to_palm: type fixed, parent iiwa_s_model_connector, child iiwa_s_model_palm, origin xyz=0 0 0.18 rpy=0 0 3.40339
- added joint iiwa_joint_1: type revolute, parent iiwa_link_0, child iiwa_link_1, origin xyz=0 0 0.1575 rpy=0 0 0, axis 0 0 1, limit lower=-2.96705972839 upper=2.96705972839 effort=300 velocity=10
- added joint iiwa_joint_2: type revolute, parent iiwa_link_1, child iiwa_link_2, origin xyz=0 0 0.2025 rpy=1.57079632679   0 3.14159265359, axis 0 0 1, limit lower=-2.09439510239 upper=2.09439510239 effort=300 velocity=10
- added joint iiwa_joint_3: type revolute, parent iiwa_link_2, child iiwa_link_3, origin xyz=0 0.2045 0 rpy=1.57079632679 0 3.14159265359, axis 0 0 1, limit lower=-2.96705972839 upper=2.96705972839 effort=300 velocity=10
- added joint iiwa_joint_4: type revolute, parent iiwa_link_3, child iiwa_link_4, origin xyz=0 0 0.2155 rpy=1.57079632679 0 0, axis 0 0 1, limit lower=-2.09439510239 upper=2.09439510239 effort=300 velocity=10
- added joint iiwa_joint_5: type revolute, parent iiwa_link_4, child iiwa_link_5, origin xyz=0 0.1845 0 rpy=-1.57079632679 3.14159265359 0, axis 0 0 1, limit lower=-2.96705972839 upper=2.96705972839 effort=300 velocity=10
- added joint iiwa_joint_6: type revolute, parent iiwa_link_5, child iiwa_link_6, origin xyz=0 0 0.2155 rpy=1.57079632679 0 0, axis 0 0 1, limit lower=-2.09439510239 upper=2.09439510239 effort=300 velocity=10
- added joint iiwa_joint_7: type revolute, parent iiwa_link_6, child iiwa_link_7, origin xyz=0 0.081 0 rpy=-1.57079632679 3.14159265359 0, axis 0 0 1, limit lower=-3.05432619099 upper=3.05432619099 effort=300 velocity=10
- added joint iiwa_joint_ee: type fixed, parent iiwa_link_7, child iiwa_link_ee, origin xyz=0 0 0.045 rpy=0 0 0
- added joint iiwa_link_ee_to_connector: type fixed, parent iiwa_link_ee, child iiwa_s_model_connector, origin xyz=0 0 0.02 rpy=0 0 0
- added joint iiwa_s_model_joint_1: type fixed, parent iiwa_s_model_palm, child iiwa_s_model_finger_1, origin xyz=0 0 0 rpy=0 0 0
- added joint iiwa_s_model_joint_2: type fixed, parent iiwa_s_model_palm, child iiwa_s_model_finger_2, origin xyz=0 0 0 rpy=0 0 0
- added joint iiwa_s_model_joint_3: type fixed, parent iiwa_s_model_palm, child iiwa_s_model_finger_3, origin xyz=0 0 0 rpy=0 0 0
- added joint world_iiwa_joint: type fixed, parent world, child iiwa_link_0, origin xyz=0 0 0.0 rpy=0 0 0
