Commit message: Add table on which iiwa is mounted on.

File: urdf/iiwa14_touch_s_model.urdf.xacro (robot description, xacro)
@@ -8,10 +8,97 @@
   <!--<xacro:include filename="$(find robotiq_s_model_visualization)/cfg/s-model_articulated_macro.xacro" />-->
   <xacro:include filename="$(find robotiq_s_model_visualization)/cfg/s-model_mesh_macro.xacro" />
-  <!-- Fix to world just for testing -->
+  <material name="wood">
+    <color rgba="0.89 0.58 0.47 0.3"/>
+  </material>
+  <material name="aluminium">
+    <color rgba="0.7 0.7 0.7 0.4"/>
+  </material>
   <link name="world"/>
+  <joint name="world_table" type="fixed">
+    <parent link="world" />
+    <child link="table" />
+  </joint>
+  <!-- Create table on which iiwa is standing -->
+  <link name="table">
+    <inertial>
+      <origin xyz="0.0 0.0 0.5" rpy="0 0 0"/>
+      <mass value="15"/>
+      <inertia ixx="0.05"  ixy="0"  ixz="0" iyy="0.06" iyz="0" izz="0.03" />
+    </inertial>
+    <visual>
+      <origin xyz="0 0 0.70" rpy="0 0 0"/>
+      <geometry>
+        <box size="1.5 1.5 0.04"/>
+      </geometry>
+      <material name="wood"/>
+    </visual>
+    <visual>
+      <origin xyz="0.66 0.66 0.34" rpy="0 0 0"/>
+      <geometry>
+        <box size="0.08 0.08 0.68"/>
+      </geometry>
+      <material name="aluminium"/>
+    </visual>
+    <visual>
+      <origin xyz="-0.66 0.66 0.34" rpy="0 0 0"/>
+      <geometry>
+        <box size="0.08 0.08 0.68"/>
+      </geometry>
+      <material name="aluminium"/>
+    </visual>
+    <visual>
+      <origin xyz="0.66 -0.66 0.34" rpy="0 0 0"/>
+      <geometry>
+        <box size="0.08 0.08 0.68"/>
+      </geometry>
+      <material name="aluminium"/>
+    </visual>
+    <visual>
+      <origin xyz="-0.66 -0.66 0.34" rpy="0 0 0"/>
+      <geometry>
+        <box size="0.08 0.08 0.68"/>
+      </geometry>
+      <material name="aluminium"/>
+    </visual>
+    <collision>
+      <origin xyz="0 0 0.70" rpy="0 0 0"/>
+      <geometry>
+        <box size="1.5 1.5 0.04"/>
+      </geometry>
+      <material name="wood"/>
+    </collision>
+    <collision>
+      <origin xyz="0.66 0.66 0.34" rpy="0 0 0"/>
+      <geometry>
+        <box size="0.08 0.08 0.68"/>
+      </geometry>
+      <material name="aluminium"/>
+    </collision>
+    <collision>
+      <origin xyz="-0.66 0.66 0.34" rpy="0 0 0"/>
+      <geometry>
+        <box size="0.08 0.08 0.68"/>
+      </geometry>
+      <material name="aluminium"/>
+    </collision>
+    <collision>
+      <origin xyz="0.66 -0.66 0.34" rpy="0 0 0"/>
+      <geometry>
+        <box size="0.08 0.08 0.68"/>
+      </geometry>
+      <material name="aluminium"/>
+    </collision>
+    <collision>
+      <origin xyz="-0.66 -0.66 0.34" rpy="0 0 0"/>
+      <geometry>
+        <box size="0.08 0.08 0.68"/>
+      </geometry>
+      <material name="aluminium"/>
+    </collision>
+  </link>
   <!--iiwa-->
   <!-- PositionJointInterface -->
-  <xacro:iiwa14 hardware_interface="$(arg hardware_interface)" robot_name="$(arg robot_name)" parent="world">
-    <origin xyz="0 0 0.0" rpy="0 0 0" />
+  <xacro:iiwa14 hardware_interface="$(arg hardware_interface)" robot_name="$(arg robot_name)" parent="table">
+    <origin xyz="0 0 0.72" rpy="0 0 0" />
   </xacro:iiwa14>
   <joint name="$(arg robot_name)_link_ee_to_connector"  type="fixed">

File: urdf/robot.urdf (robot description, URDF)
Before this commit: robot iiwa_s_m, 15 links, 14 joints
Links:
- added link table, mass 15; collision box size=0.08 0.08 0.68; collision box size=0.08 0.08 0.68
Joints:
- removed joint world_iiwa_joint
- added joint table_iiwa_joint: type fixed, parent table, child iiwa_link_0, origin xyz=0 0 0.72 rpy=0 0 0
- added joint world_table: type fixed, parent world, child table
