Commit message: Add dummy link that represents the world frame as Sunrise uses it and set tool parameter to 'gripper' when uploading the robot model.

File: iiwa14_s_model_description/urdf/iiwa14_touch_s_model.urdf.xacro (robot description, xacro)
@@ -171,3 +171,9 @@
   <xacro:s-model_mesh prefix="$(arg robot_name)_s_model_">
   </xacro:s-model_mesh>
+  <joint name="world_sunrise_world" type="fixed">
+    <origin xyz="$(arg origin_xyz)" rpy="0 0 0" />
+    <parent link="world" />
+    <child link="sunrise_world" />
+  </joint>
+  <link name="sunrise_world" />
 </robot>

Commit message: Adjust mounted robot height.

File: iiwa14_s_model_description/urdf/iiwa14_touch_s_model.urdf.xacro (robot description, xacro)
@@ -10,5 +10,5 @@
   <xacro:arg name="hardware_interface" default="PositionJointInterface"/>
   <xacro:arg name="robot_name" default="iiwa"/>
-  <xacro:arg name="origin_xyz" default="0 0 1.71"/><!-- 0 0 1.71 -->
+  <xacro:arg name="origin_xyz" default="0 0 1.735"/><!-- 0 0 1.71 -->
   <xacro:arg name="origin_rpy" default="0 1.570796327 0"/>
   <!-- Fix to world just for testing -->
@@ -166,5 +166,5 @@
       <parent link="$(arg robot_name)_s_model_connector"/>
       <child link="$(arg robot_name)_s_model_palm"/>
-      <origin xyz="0 0 0.18" rpy="0 0 ${3.14159+0.2618}"/>
+      <origin xyz="0 0 0.18" rpy="0 0 0"/>
     </joint>
   </xacro:unless>
